Commit message: update

File: install/doosan_m0609_description/share/doosan_m0609_description/urdf/m0609.white.urdf (robot description, URDF)
Before this commit: robot m0609, 8 links, 7 joints
Links:
- link base_link: geometry visual mesh filename=package://doosan_m0609_description/meshes/m0609_white/MF060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 scale=0.001 0.001 0.001
- link link_1: geometry visual mesh filename=package://doosan_m0609_description/meshes/m0609_white/MF060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 scale=0.001 0.001 0.001
- link link_2: geometry visual mesh filename=package://doosan_m0609_description/meshes/m0609_white/MF060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 scale=0.001 0.001 0.001; visual mesh filename=package://doosan_m0609_description/meshes/m0609_white/MF060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 scale=0.001 0.001 0.001
- link link_3: geometry visual mesh filename=package://doosan_m0609_description/meshes/m0609_white/MF060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 scale=0.001 0.001 0.001
- link link_4: geometry visual mesh filename=package://doosan_m0609_description/meshes/m0609_white/MF060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 scale=0.001 0.001 0.001; visual mesh filename=package://doosan_m0609_description/meshes/m0609_white/MF060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 scale=0.001 0.001 0.001
- link link_5: geometry visual mesh filename=package://doosan_m0609_description/meshes/m0609_white/MF060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 scale=0.001 0.001 0.001
- link link_6: geometry visual mesh filename=package://doosan_m0609_description/meshes/m0609_white/MF060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 scale=0.001 0.001 0.001
